File: RPi_Hat.kicad_pcb (KiCad board)
At the start: 2 copper layers, 65 x 56.5 mm, 21 parts, among them IC1 0.96_I2C_OLED, IC2 7406, IC3 I2C LC, J1 RPi_GPIO, SW1 Select, SW2 Up, SW3 Down, SW4 Exit, SW5 Add Disk

Commit message: Revision B PCB layout
Parts:
- IC1: footprint IIC_OLED:0.91_I2C_OLED -> IIC_OLED:0.96_I2C_OLED
- IEC_1: renamed from IEC #1
- IEC_2: renamed from IEC #2
- moved IC1 22.0 mm to (43.8, 36.8)
- moved C1 18.7 mm to (33.1, 58.6)
- moved IC2 18.7 mm to (37.0, 65.0)
- moved BZ1 18.4 mm to (61.1, 57.4), turned to 0 degrees
- moved R1 12.5 mm to (68.1, 39.6)
- moved R2 12.5 mm to (64.3, 49.7)
- moved R3 12.5 mm to (60.4, 49.7)
- moved IC3 7.73 mm to (43.2, 48.3), turned to 90 degrees
Routing:
- net RPI_CLK_OUT: track 16.8 -> 60.4 mm
- net Net-(D1-Pad1): track 24.9 -> 54.6 mm
- net C64_DATA: track 78.7 -> 108.4 mm, vias 1 -> 5
- net RPI_DATA_OUT: track 28.5 -> 54.6 mm
- net C64_CLK: track 73.2 -> 98.2 mm, vias 3 -> 5
- net RPI_ATN: track 50.3 -> 27.7 mm, vias 2 -> 0
- net RPI_CLK_IN: track 73.4 -> 54.2 mm, vias 2 -> 3
- net RPI_SND: track 13.5 -> 31.6 mm
- net IN_SW4: track 59.7 -> 77.0 mm, vias 2 -> 0
- net I2C_SCL: track 25.7 -> 13.0 mm, vias 0 -> 2
- net C64_ATN: track 61.3 -> 51.9 mm, vias 1 -> 3
- net C64_RST: track 49.4 -> 58.1 mm, vias 0 -> 5
- net +3V3: track 33.3 -> 39.5 mm, vias 0 -> 2
- net RPI_RST: track 54.5 -> 60.4 mm, vias 2 -> 5
- net +5V: track 76.6 -> 71.3 mm, vias 0 -> 1
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Other:
- board text added: "PCB Rev. B"
- board text removed: "PCB Rev. A"

Commit message: Revision B gerber export
Parts:
- added IC4: 0.96_I2C_OLED, IIC_OLED:0.91_I2C_OLED, F.Cu at (48.4, 45.9)
Routing:
- net I2C_SCL: track 13.0 -> 23.2 mm, vias 2 -> 4
- net I2C_SDA: track 20.0 -> 29.3 mm
- net RPI_CLK_OUT: track 60.4 -> 69.1 mm
- net RPI_DATA_OUT: track 54.6 -> 61.5 mm
- net +3V3: track 39.5 -> 42.8 mm
- net +5V: track 71.3 -> 72.4 mm

Commit message: Bumped revision number
Other:
- board text added: "PCB Rev. C"
- board text removed: "PCB Rev. B"
Changed lines of the file:
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@@
   )
   (setup
-    (last_trace_width 0.01)
+    (last_trace_width 0.25)
     (user_trace_width 0.01)
     (user_trace_width 0.02)
@@
       (effects (font (size 1 1) (thickness 0.15)))
     )
-    (fp_text value 7406 (at 3.81 17.57 90) (layer F.Fab)
+    (fp_text value 7406 (at 3.81 17.57 90) (layer F.SilkS)
       (effects (font (size 1 1) (thickness 0.15)))
     )
@@
     (descr "Resistor, Axial_DIN0207 series, Axial, Horizontal, pin pitch=10.16mm, 0.25W = 1/4W, length*diameter=6.3*2.5mm^2, http://cdn-reichelt.de/documents/datenblatt/B400/1_4W%23YAG.pdf")
     (tags "Resistor Axial_DIN0207 series Axial Horizontal pin pitch 10.16mm 0.25W = 1/4W length 6.3mm diameter 2.5mm")
-    (fp_text reference R1 (at 5.08 0 360) (layer F.SilkS)
-      (effects (font (size 1 1) (thickness 0.15)))
-    )
-    (fp_text value 100 (at 5.08 2.31 270) (layer F.Fab)
+    (fp_text reference R1 (at 3.175 0 360) (layer F.SilkS)
+      (effects (font (size 1 1) (thickness 0.15)))
+    )
+    (fp_text value 100 (at 5.08 2.31 270) (layer F.SilkS) hide
       (effects (font (size 1 1) (thickness 0.15)))
     )
@@
     (descr "Resistor, Axial_DIN0207 series, Axial, Horizontal, pin pitch=10.16mm, 0.25W = 1/4W, length*diameter=6.3*2.5mm^2, http://cdn-reichelt.de/documents/datenblatt/B400/1_4W%23YAG.pdf")
     (tags "Resistor Axial_DIN0207 series Axial Horizontal pin pitch 10.16mm 0.25W = 1/4W length 6.3mm diameter 2.5mm")
-    (fp_text reference R2 (at 5.08 0 180) (layer F.SilkS)
-      (effects (font (size 1 1) (thickness 0.15)))
-    )
-    (fp_text value 1K (at 5.08 2.31 90) (layer F.Fab)
+    (fp_text reference R2 (at 6.985 0 180) (layer F.SilkS)
+      (effects (font (size 1 1) (thickness 0.15)))
+    )
+    (fp_text value 1K (at 5.08 2.31 90) (layer F.SilkS) hide
       (effects (font (size 1 1) (thickness 0.15)))
     )
@@
     (descr "Resistor, Axial_DIN0207 series, Axial, Horizontal, pin pitch=10.16mm, 0.25W = 1/4W, length*diameter=6.3*2.5mm^2, http://cdn-reichelt.de/documents/datenblatt/B400/1_4W%23YAG.pdf")
     (tags "Resistor Axial_DIN0207 series Axial Horizontal pin pitch 10.16mm 0.25W = 1/4W length 6.3mm diameter 2.5mm")
-    (fp_text reference R3 (at 5.08 0 180) (layer F.SilkS)
-      (effects (font (size 1 1) (thickness 0.15)))
-    )
-    (fp_text value 1K (at 5.08 2.31 90) (layer F.Fab)
+    (fp_text reference R3 (at 6.985 0 180) (layer F.SilkS)
+      (effects (font (size 1 1) (thickness 0.15)))
+    )
+    (fp_text value 1K (at 5.08 2.31 90) (layer F.SilkS) hide
       (effects (font (size 1 1) (thickness 0.15)))
     )
@@
       (net 6 I2C_SDA))
   )
-  (gr_text "PCB\nRev. B" (at 27.305 41.91 270) (layer F.SilkS)
+  (gr_text "PCB\nRev. C" (at 27.305 41.91 270) (layer F.SilkS)
     (effects (font (size 1.5 1.5) (thickness 0.3)))
   )
@@
     (effects (font (size 1.5 1.5) (thickness 0.3)) (justify left mirror))
   )
-  (gr_text Pi1541 (at 39.37 43.434) (layer B.SilkS)
+  (gr_text Pi1541 (at 50.92 70.7) (layer B.SilkS)
     (effects (font (size 4 4) (thickness 0.4) italic) (justify mirror))
   )
@@
   (via (at 35.68 36.41) (size 0.6) (drill 0.4) (layers F.Cu B.Cu) (net 5))
   (segment (start 36.95 35.14) (end 35.68 36.41) (width 0.25) (layer F.Cu) (net 5))
-  (segment (start 34.41 42.76) (end 33.775 43.395) (width 0.25) (layer F.Cu) (net 5) (status 800000))
-  (segment (start 33.775 43.395) (end 33.14 43.395) (width 0.25) (layer F.Cu) (net 5) (status C00000))
+  (segment (start 34.41 42.76) (end 33.775 43.395) (width 0.25) (layer F.Cu) (net 5))
+  (segment (start 33.775 43.395) (end 33.14 43.395) (width 0.25) (layer F.Cu) (net 5))
   (segment (start 45.685 39.52) (end 45.685 37.525) (width 0.25) (layer F.Cu) (net 5))
   (segment (start 38.22 36.41) (end 41.395 36.41) (width 0.25) (layer F.Cu) (net 5))
@@
   (segment (start 45.685 37.525) (end 45.205 37.045) (width 0.25) (layer F.Cu) (net 5))
   (segment (start 36.95 33.85) (end 36.945 33.845) (width 0.25) (layer F.Cu) (net 5))
-  (segment (start 33.14 40.855) (end 33.14 39.585) (width 0.25) (layer F.Cu) (net 6) (status 400000))
+  (segment (start 33.14 40.855) (end 33.14 39.585) (width 0.25) (layer F.Cu) (net 6))
   (segment (start 31.87 38.315) (end 31.87 36.41) (width 0.25) (layer F.Cu) (net 6))
   (segment (start 31.87 36.41) (end 32.505 35.775) (width 0.25) (layer F.Cu) (net 6))
@@
   (segment (start 35.68 41.49) (end 36.315 40.855) (width 0.25) (layer F.Cu) (net 14))
   (segment (start 35.68 45.3) (end 35.68 41.49) (width 0.25) (layer F.Cu) (net 14))
-  (segment (start 33.14 45.935) (end 35.045 45.935) (width 0.25) (layer F.Cu) (net 14) (status 400000))
+  (segment (start 33.14 45.935) (end 35.045 45.935) (width 0.25) (layer F.Cu) (net 14))
   (segment (start 43.3 51.65) (end 43.3 53.22) (width 0.25) (layer F.Cu) (net 14))
   (segment (start 42.03 50.38) (end 43.3 51.65) (width 0.25) (layer F.Cu) (net 14))
@@
   (segment (start 31.865 35.145) (end 31.235 35.775) (width 0.25) (layer F.Cu) (net 14))
   (segment (start 31.865 33.845) (end 31.865 35.145) (width 0.25) (layer F.Cu) (net 14))
-  (segment (start 31.87 45.935) (end 33.14 45.935) (width 0.25) (layer F.Cu) (net 14) (status 800000))
+  (segment (start 31.87 45.935) (end 33.14 45.935) (width 0.25) (layer F.Cu) (net 14))
   (segment (start 31.235 45.3) (end 31.87 45.935) (width 0.25) (layer F.Cu) (net 14))
   (segment (start 43.145 39.74) (end 43.145 39.52) (width 0.25) (layer F.Cu) (net 14))
